Commit message: Added CAD meshes to the mini_Pi and maze world with the launch file that starts RViz and Gazebo.

File: xacro/macros/caster.xacro (robot description, xacro)
@@ -36,4 +36,5 @@
       <child link="${name}_yaw_link"/>
       <axis xyz="0 0 1"/>
+      <dynamics damping="0.8" friction="0.0"/>
     </joint>
     <!-- Caster Wheel Link (Roll) -->
@@ -70,4 +71,5 @@
       <child link="${name}_roll_link"/>
       <axis xyz="1 0 0"/>
+      <dynamics damping="0.02" friction="0.0"/>
     </joint>
     <!-- Caster Wheel Link (Pitch) -->
@@ -104,4 +106,5 @@
       <child link="${name}_pitch_link"/>
       <axis xyz="0 1 0"/>
+      <dynamics damping="0.05" friction="0.0"/>
     </joint>
   </xacro:macro>

File: xacro/macros/shapes.xacro (robot description, xacro)
@@ -56,4 +56,18 @@
           <cylinder radius="${radius}" length="${length}" />
         </geometry>
+        <surface>
+          <friction>
+            <ode>
+              <mu>1.5</mu>
+              <mu2>1.5</mu2>
+            </ode>
+          </friction>
+          <contact>
+            <ode>
+              <kp>1e6</kp>
+              <kd>1.0</kd>
+            </ode>
+          </contact>
+        </surface>
       </collision>
       <inertial>

File: xacro/mini_pi.xacro (robot description, xacro)
@@ -3,7 +3,10 @@
   <!-- Colors -->
   <xacro:include filename="$(find mini_pi_description)/xacro/materials/materials.xacro"/>
-  <!-- Shapes & Caster -->
+  <!-- Shapes & Caster,Sensor,Chassis -->
   <xacro:include filename="$(find mini_pi_description)/xacro/macros/shapes.xacro"/>
+  <xacro:include filename="$(find mini_pi_description)/xacro/macros/wheel.xacro"/>
   <xacro:include filename="$(find mini_pi_description)/xacro/macros/caster.xacro"/>
+  <xacro:include filename="$(find mini_pi_description)/xacro/macros/ultrasonic_sensor.xacro"/>
+  <xacro:include filename="$(find mini_pi_description)/xacro/macros/chassis.xacro"/>
   <!-- Robot Parts -->
   <xacro:include filename="$(find mini_pi_description)/xacro/parts/params.xacro"/>
@@ -67,4 +70,23 @@
       <state_interface name="velocity"/>
     </joint>
+    <!-- CASTER JOINTS: state-only (passive) -->
+    <joint name="front_caster_yaw_joint">
+      <state_interface name="position"/>
+    </joint>
+    <joint name="front_caster_roll_joint">
+      <state_interface name="position"/>
+    </joint>
+    <joint name="front_caster_pitch_joint">
+      <state_interface name="position"/>
+    </joint>
+    <joint name="back_caster_yaw_joint">
+      <state_interface name="position"/>
+    </joint>
+    <joint name="back_caster_roll_joint">
+      <state_interface name="position"/>
+    </joint>
+    <joint name="back_caster_pitch_joint">
+      <state_interface name="position"/>
+    </joint>
   </ros2_control>
   <!-- ==== Gazebo plugin ==== -->

File: xacro/parts/chassis.xacro (robot description, xacro)
@@ -2,10 +2,9 @@
 <robot xmlns:xacro="http://www.ros.org/wiki/xacro" name="mini_pi">
   <xacro:macro name="mini_pi_chassis" params="parent">
-    <xacro:square_link
+    <xacro:chassis
       name="chassis"
       size_x="${base_size_x}"
       size_y="${base_size_y}"
       size_z="${base_size_z}"
-      material="Red"
       mass="${base_mass}"
       parent_link="${parent}"

File: xacro/parts/sensors_ultrasonic.xacro (robot description, xacro)
@@ -6,10 +6,6 @@
   <xacro:property name="ULTRA_LEFT"  value="0       0.0485  0.0300  0  0  1.5708" />
   <xacro:macro name="mini_pi_ultrasonic" params="parent">
-    <xacro:square_link
+    <xacro:ultrasonic_sensor
     name="ultrasonic_sensor_1"
-    size_x="0.0135"
-    size_y="0.045"
-    size_z="0.0165"
-    material="Green"
     mass="0.001"
     parent_link="${parent}"
@@ -17,10 +13,6 @@
     rpy="0 0 0"
     joint_type="fixed"/>
-    <xacro:square_link
+    <xacro:ultrasonic_sensor
     name="ultrasonic_sensor_2"
-    size_x="0.0135"
-    size_y="0.045"
-    size_z="0.0165"
-    material="Green"
     mass="0.001"
     parent_link="${parent}"
@@ -28,10 +20,6 @@
     rpy="0 0 4.7123"
     joint_type="fixed"/>
-    <xacro:square_link
+    <xacro:ultrasonic_sensor
     name="ultrasonic_sensor_3"
-    size_x="0.0135"
-    size_y="0.045"
-    size_z="0.0165"
-    material="Green"
     mass="0.001"
     parent_link="${parent}"
@@ -39,10 +27,6 @@
     rpy="0 0 3.14159"
     joint_type="fixed"/>
-    <xacro:square_link
+    <xacro:ultrasonic_sensor
     name="ultrasonic_sensor_4"
-    size_x="0.0135"
-    size_y="0.045"
-    size_z="0.0165"
-    material="Green"
     mass="0.001"
     parent_link="${parent}"

File: xacro/parts/wheels.xacro (robot description, xacro)
@@ -2,9 +2,8 @@
 <robot xmlns:xacro="http://www.ros.org/wiki/xacro" name="mini_pi">
   <xacro:macro name="mini_pi_wheels" params="parent">
-    <xacro:cylinder_link
+    <xacro:wheel
       name="wheel_right"
       radius="${wheel_radius}"
       length="${wheel_width}"
-      material="Black"
       mass="${wheel_mass}"
       parent_link="${parent}"
@@ -13,9 +12,8 @@
       joint_type="continuous"
       axis="0 1 0"/>
-    <xacro:cylinder_link
+    <xacro:wheel
       name="wheel_left"
       radius="${wheel_radius}"
       length="${wheel_width}"
-      material="Black"
       mass="${wheel_mass}"
       parent_link="${parent}"
